Commit message: Changed to 5 DOF, changed names of joints to match new urdf and commented static tf publisher to not interfer with new rviz

File: arm_control/description/ros2_control/hardware_ros2_control.xacro (robot description, xacro)
@@ -81,28 +81,13 @@
         <state_interface name="temperature"/>
       </joint>
-      <!-- FIXED: joint6 not joint_6 -->
-      <joint name="joint6">
-        <param name="id">6</param>
-        <param name="type">pos</param>
-        <param name="offset">3.141592</param>
-        <param name="gear_ratio">1.0</param> <!-- gear ratio -->
-        <command_interface name="position">
-          <param name="min">-2.09</param>
-          <param name="max">2.09</param>
-        </command_interface>
-        <state_interface name="position"/>
-        <state_interface name="velocity"/>
-        <state_interface name="torque"/>
-        <state_interface name="temperature"/>
-      </joint>
       <!-- Gripper with MATCHING interfaces -->
-      <joint name="gripper_controller">
+      <joint name="gripper1">
         <param name="id">7</param>
         <param name="type">pos</param>
         <param name="offset">3.141592</param>
-        <param name="gear_ratio">1.75</param> <!-- gear ratio -->
+        <param name="gear_ratio">5.2</param> <!-- gear ratio -->
         <command_interface name="position">
-          <param name="min">-0.4</param>  <!-- Match main PC limits -->
-          <param name="max">0.6</param>
+          <param name="min">-0.3</param>  <!-- Match main PC limits -->
+          <param name="max">0.3</param>
         </command_interface>
         <state_interface name="position"/>

File: arm_control/description/urdf/test.urdf.xacro (robot description, xacro)
@@ -1,11 +1,8 @@
 <?xml version="1.0"?>
 <robot xmlns:xacro="http://www.ros.org/wiki/xacro" name="test">
-  <!-- Include the ros2_control definition -->
   <xacro:include filename="$(find arm_control)/description/ros2_control/hardware_ros2_control.xacro"/>
-  <!-- Materials -->
   <material name="grey"><color rgba="0.5 0.5 0.5 1"/></material>
   <material name="blue"><color rgba="0.1 0.1 0.8 1"/></material>
   <material name="red"><color rgba="0.8 0.1 0.1 1"/></material>
-  <!-- Base Link -->
   <link name="base_link">
     <visual>
@@ -14,5 +11,4 @@
     </visual>
   </link>
-  <!-- ODrive Links (joints 0-2) -->
   <link name="odrive_link_1">
     <visual>
@@ -36,5 +32,4 @@
     </visual>
   </link>
-  <!-- Waveshare Servo Links (joints 3-5) -->
   <link name="servo_link_1">
     <visual>
@@ -49,11 +44,4 @@
     </visual>
   </link>
-  <link name="servo_link_3">
-    <visual>
-      <geometry><cylinder length="0.06" radius="0.02"/></geometry>
-      <material name="red"/>
-    </visual>
-  </link>
-  <!-- Gripper Link -->
   <link name="gripper_link">
       <visual>
@@ -67,6 +55,4 @@
       </collision>
   </link>
-  <!-- FIXED JOINT LIMITS TO MATCH MAIN PC -->
-  <!-- Joint 1: MATCHED limits -->
   <joint name="joint1" type="revolute">
     <parent link="base_link"/>
@@ -76,5 +62,4 @@
     <limit effort="10" lower="-3.12" upper="3.12" velocity="1"/>
   </joint>
-  <!-- Joint 2: MATCHED limits -->
   <joint name="joint2" type="revolute">
     <parent link="odrive_link_1"/>
@@ -84,5 +69,4 @@
     <limit effort="10" lower="-1.05" upper="1.92" velocity="1"/>
   </joint>
-  <!-- Joint 3: MATCHED limits -->
   <joint name="joint3" type="revolute">
     <parent link="odrive_link_2"/>
@@ -92,5 +76,4 @@
     <limit effort="10" lower="-2.27" upper="2.27" velocity="1"/>
   </joint>
-  <!-- Joint 4: MATCHED limits -->
   <joint name="joint4" type="revolute">
     <parent link="base_link"/>
@@ -100,5 +83,4 @@
     <limit effort="1" lower="-2.09" upper="2.09" velocity="1"/>
   </joint>
-  <!-- Joint 5: MATCHED limits -->
   <joint name="joint5" type="revolute">
     <parent link="servo_link_1"/>
@@ -108,19 +90,10 @@
     <limit effort="1" lower="-2.09" upper="2.09" velocity="1"/>
   </joint>
-  <!-- Joint 6: MATCHED limits -->
-  <joint name="joint6" type="revolute">
-    <parent link="servo_link_2"/>
-    <child link="servo_link_3"/>
-    <origin xyz="0 0 0.1"/>
-    <axis xyz="1 0 0"/>
-    <limit effort="1" lower="-2.09" upper="2.09" velocity="1"/>
-  </joint>
-  <!-- Gripper Joint: MATCHED limits -->
-  <joint name="gripper_controller" type="revolute">
-      <parent link="servo_link_3"/>
+  <joint name="gripper1" type="revolute">
+      <parent link="servo_link_2"/>
       <child link="gripper_link"/>
       <origin xyz="0 0 0.06" rpy="0 0 0"/>
       <axis xyz="0 1 0"/>
-      <limit lower="-0.6" upper="0.4" effort="5" velocity="1.0"/>
+      <limit lower="-0.3" upper="0.3" effort="1" velocity="1"/>
   </joint>
   <xacro:arm_control/>

Commit message: sensors added (tof, load cell) and general changes

File: arm_control/description/ros2_control/hardware_ros2_control.xacro (robot description, xacro)
@@ -19,4 +19,5 @@
         <state_interface name="position"/>
         <state_interface name="velocity"/>
+        <state_interface name="effort"/>
         <!-- Remove 'effort' to match main PC -->
       </joint>
@@ -24,22 +25,24 @@
         <param name="node_id">1</param>
         <param name="type">pos</param>
-        <param name="gear_ratio">295.0</param>  <!-- Match main PC gear ratio -->
+        <param name="gear_ratio">304.6</param>  <!-- Match main PC gear ratio  prev. ratio 295.00 -->
         <command_interface name="position">
-          <param name="min">-1.05</param>  <!-- Match main PC limits -->
+          <param name="min">-0.897</param>  <!-- Match main PC limits -->
           <param name="max">1.92</param>
         </command_interface>
         <state_interface name="position"/>
         <state_interface name="velocity"/>
+        <state_interface name="effort"/>
       </joint>
       <joint name="joint3">
         <param name="node_id">2</param>
         <param name="type">pos</param>
-        <param name="gear_ratio">196.87</param>  <!-- Match main PC gear ratio -->
+        <param name="gear_ratio">198.0</param>  <!-- Match main PC gear ratio -->
         <command_interface name="position">
-          <param name="min">-2.27</param>  <!-- Match main PC limits -->
-          <param name="max">2.27</param>
+          <param name="min">-1.83</param>  <!-- Match main PC limits -->
+          <param name="max">1.83</param>
         </command_interface>
         <state_interface name="position"/>
         <state_interface name="velocity"/>
+        <state_interface name="effort"/>
       </joint>
     </ros2_control>
@@ -55,5 +58,5 @@
         <param name="id">4</param>
         <param name="type">pos</param>
-        <param name="offset">3.141592</param>
+        <param name="offset">3.041592</param>
         <param name="gear_ratio">1.0</param> <!-- gear ratio -->
         <command_interface name="position">
@@ -61,4 +64,5 @@
           <param name="max">2.09</param>
         </command_interface>
+        <command_interface name="velocity"/>
         <state_interface name="position"/>
         <state_interface name="velocity"/>
@@ -68,7 +72,7 @@
       </joint>
       <joint name="joint5">
-        <param name="id">5</param>
+        <param name="id">6</param>
         <param name="type">pos</param>
-        <param name="offset">3.141592</param>
+        <param name="offset">3.181592</param>
         <param name="gear_ratio">1.0</param> <!-- gear ratio -->
         <command_interface name="position">
@@ -76,4 +80,5 @@
           <param name="max">2.09</param>
         </command_interface>
+        <command_interface name="velocity"/>
         <state_interface name="position"/>
         <state_interface name="velocity"/>

File: arm_control/description/urdf/test.urdf.xacro (robot description, xacro)
@@ -50,8 +50,4 @@
           <material name="grey"/>
       </visual>
-      <collision>
-          <geometry><box size="0.02 0.1 0.02"/></geometry>
-          <origin xyz="0 0 0.05" rpy="0 0 0"/>
-      </collision>
   </link>
   <joint name="joint1" type="revolute">
@@ -77,7 +73,7 @@
   </joint>
   <joint name="joint4" type="revolute">
-    <parent link="base_link"/>
+    <parent link="odrive_link_3"/>
     <child link="servo_link_1"/>
-    <origin xyz="0 0.1 0.1"/>
+    <origin xyz="0 0 0.3"/>
     <axis xyz="0 0 1"/>
     <limit effort="1" lower="-2.09" upper="2.09" velocity="1"/>

File: ros_waveshare/waveshare_explorer/description/urdf/single_servo.urdf.xacro (robot description, xacro)
@@ -34,5 +34,5 @@
         <origin xyz="0 0 0.025" rpy="0 0 0"/>
         <axis xyz="0 0 1"/>
-        <limit lower="-1.570796" upper="1.570796" effort="10" velocity="1.0"/>
+        <limit lower="-1.570796" upper="1.570796" effort="100" velocity="500.0"/>
     </joint>
     <!-- Instantiate the ros2_control macro -->
